Commit message: removing dependency on mimic joints

File: assets/urdf/ur5_robotiq85_gripper.urdf (robot description, URDF)
Before this commit: robot ur5, 21 links, 20 joints
Joints:
- joint robotiq_85_left_finger_tip_joint: limit lower=-3.14 upper=3.14 effort=0.1 velocity=100.0 -> lower=-3.14 upper=3.14 effort=1000 velocity=2.0; type continuous -> revolute
- joint robotiq_85_left_inner_knuckle_joint: limit lower=-3.14 upper=3.14 effort=0.1 velocity=100.0 -> lower=-3.14 upper=3.14 effort=1000 velocity=2.0; type continuous -> revolute
- joint robotiq_85_left_knuckle_joint: limit lower=0.0 upper=0.80285 effort=1000 velocity=0.5 -> lower=0.0 upper=0.80285 effort=1000 velocity=2.0
- joint robotiq_85_right_finger_tip_joint: limit lower=-3.14 upper=3.14 effort=0.1 velocity=100.0 -> lower=-3.14 upper=3.14 effort=1000 velocity=2.0; type continuous -> revolute
- joint robotiq_85_right_inner_knuckle_joint: limit lower=-3.14 upper=3.14 effort=0.1 velocity=100.0 -> lower=-3.14 upper=3.14 effort=1000 velocity=2.0; type continuous -> revolute
- joint robotiq_85_right_knuckle_joint: limit lower=-3.14 upper=3.14 effort=1000 velocity=100.0 -> lower=-3.14 upper=3.14 effort=1000 velocity=2.0; type continuous -> revolute
